File: custack-hardware/electric/battery_board.kicad_sch (KiCad schematic)
At the start: 10 parts, among them J1 XH 2.5mmピッチ 2極 オス AWG24, Q1 MOSFET P-CH 20V 6A SOT23F, SW1 12V 100mA

Commit message: 型番確定作業途中
Parts:
- J1: value XH 2.5mmピッチ 2極 オス AWG24 -> XH 2.5mmピッチ 2極 オス AWG22
Other:
- note added: "18350バッテリ 3.7V(MAX 4.2V) 3A 1400mAh"
- note added: "Gate印加電圧 3.7V~4.2V V_{GS} = -4.2V~-3.7V V_{GSS} = ±8V"
- note added: "R_{DS(ON)} = 29.8mohm @V_{GS} = -4.5V 3A^2 * 0.0298ohm = 0.2682W 125°C/W * 0.2682W = 33.525°C"
- note removed: "18350バッテリ 3.7V(MAX 4.7V) 3A 1400mAh"
- note removed: "Gate印加電圧 3.7V~4.7V V_{GS} = -4.7V~-3.7V V_{GSS} = ±8V"
- note removed: "R_{DS(ON)} = 29.8mohm @V_{GS} = -4.5V 3A^2 * 0.0298ohm = 0.2682W 125℃/W * 0.2682W = 33.525°C"
Changed lines of the file:
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@@
 		)
 	)
-	(text "R_{DS(ON)} = 29.8mohm @V_{GS} = -4.5V\n3A^2 * 0.0298ohm = 0.2682W\n125℃/W * 0.2682W = 33.525°C"
+	(text "R_{DS(ON)} = 29.8mohm @V_{GS} = -4.5V\n3A^2 * 0.0298ohm = 0.2682W\n125°C/W * 0.2682W = 33.525°C"
 		(exclude_from_sim no)
 		(at 138.684 50.038 0)
@@
 		)
 	)
-	(text "Gate印加電圧\n3.7V~4.7V\nV_{GS} = -4.7V~-3.7V\nV_{GSS} = ±8V\n"
+	(text "Gate印加電圧\n3.7V~4.2V\nV_{GS} = -4.2V~-3.7V\nV_{GSS} = ±8V\n"
 		(exclude_from_sim no)
 		(at 114.046 47.498 0)
@@
 		)
 	)
-	(text "18350バッテリ\n3.7V(MAX 4.7V) 3A\n1400mAh"
+	(text "18350バッテリ\n3.7V(MAX 4.2V) 3A\n1400mAh"
 		(exclude_from_sim no)
 		(at 32.258 38.1 0)
@@
 			)
 		)
-		(property "Value" "XH 2.5mmピッチ 2極 オス AWG24"
+		(property "Value" "XH 2.5mmピッチ 2極 オス AWG22"
 			(at 190.52 36.8299 0)
 			(show_name no)

Commit message: electric circut complete
Parts:
- removed BT1: 18350 2S, My_Custom:18350_2S_custom, symbol My_Customy:18350_2S
- removed C1: 220µF 25V 105°C, Capacitor_SMD:CP_Elec_8x10, symbol My_Device:C_Polarized_Small
- removed C2: 10µF 25V X5R, Capacitor_SMD:C_0603_1608Metric, symbol My_Device:C_Small
- removed D4: 20V 3A Vf=500mV, Diode_SMD:D_SMA, symbol My_Device:D_Small
- removed Q1: MOSFET P-CH 20V 6A SOT23F, Package_TO_SOT_SMD:SOT-23, symbol Device:Q_PMOS
- added BT1: 18350 2S, My_Custom:18350_2S_custom, symbol My_Custom:18350_2S
- added C1: 10µF 25V X5R, Capacitor_SMD:C_0603_1608Metric, symbol My_Device:C_Small
- added C2: 220µF 25V 105°C, Capacitor_SMD:CP_Elec_8x10, symbol My_Device:C_Polarized_Small
- added D1: 20V 3A Vf=500mV, Diode_SMD:D_SMA, symbol My_Device:D_Small
- added Q1: MOSFET P-CH 20V 6A SOT23F, Package_TO_SOT_SMD:SOT-23, symbol My_Device:Q_PMOS
Connections:
- net GND: now also J1.1 (Pin_1), BT1.4 (-), C1.1, C2.2; no longer J1.2 (Pin_2)
- net at F1.1: now also D1.1 (K)
- net +BATT: now reaches F1.2
- net +BATT: now also R1.1, Q1.3 (D)
- net at R1.2, R2.1: now also Q1.1 (G)
- new net: BT1.1 (+), D1.2 (A)
- new net: BT1.2 (-), BT1.3 (+)
- new net +VSW: C1.2, C2.1, J1.2 (Pin_2), Q1.2 (S)
- no-connect marks 0 -> 1
