File: custack-hardware/electric/battery_board.kicad_sch (KiCad schematic)
At the start: 10 parts, among them J1 XH 2.5mmピッチ 2極 オス AWG22, Q1 MOSFET P-CH 20V 6A SOT23F, SW1 12V 100mA

Commit message: complete electric board design
Connections:
- net +BATT: now also Q1.2 (S); no longer Q1.3 (D)
- net +VSW: now also Q1.3 (D); no longer Q1.2 (S)
Changed lines of the file:
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@@
 	(text "Source"
 		(exclude_from_sim no)
-		(at 145.034 79.248 0)
+		(at 145.288 71.628 0)
 		(effects
 			(font
@@
 	(text "Drain"
 		(exclude_from_sim no)
-		(at 146.558 71.882 0)
+		(at 146.558 80.264 0)
 		(effects
 			(font
@@
 	)
 	(junction
-		(at 151.13 109.22)
-		(diameter 0)
-		(color 0 0 0 0)
-	)
-	(junction
-		(at 127 76.2)
+		(at 151.13 68.58)
 		(diameter 0)
 		(color 0 0 0 0)
@@
 	)
 	(junction
-		(at 151.13 68.58)
+		(at 151.13 109.22)
+		(diameter 0)
+		(color 0 0 0 0)
+	)
+	(junction
+		(at 127 76.2)
 		(diameter 0)
 		(color 0 0 0 0)
@@
 		(lib_id "My_Device:Q_PMOS")
 		(at 148.59 76.2 0)
+		(mirror x)
 		(unit 1)
 		(body_style 1)
@@
 		(in_pos_files yes)
 		(dnp no)
-		(fields_autoplaced yes)
 		(property "Reference" "Q1"
-			(at 154.94 73.6599 0)
+			(at 154.94 78.7401 0)
 			(show_name no)
 			(do_not_autoplace no)
@@
 		)
 		(property "Value" "MOSFET P-CH 20V 6A SOT23F"
-			(at 154.94 76.1999 0)
+			(at 154.94 76.2001 0)
 			(show_name no)
 			(do_not_autoplace no)
@@
 		)
 		(property "Footprint" "Package_TO_SOT_SMD:SOT-23"
-			(at 153.67 73.66 0)
+			(at 153.67 78.74 0)
 			(hide yes)
 			(show_name no)
@@
 		)
 		(property "型式" "SSM3J328R,LF"
-			(at 154.94 78.7399 0)
-			(show_name no)
-			(do_not_autoplace no)
+			(at 154.94 73.6601 0)
+			(show_name no)
+			(do_not_autoplace no)
