File: custack-hardware/electric/custack-electric.kicad_sch (KiCad schematic)
At the start: 24 parts, among them J1 Conn_01x02, J2 Conn_01x02, J4 Conn_02x15_Odd_Even, Q1 Q_PMOS, Q2 Q_NMOS, SW1 SW_Slide_2C, U1 TPS562200DDCR

Commit message: 電子回路設計が一旦完成
Parts:
- removed BT1, BT2: ***, symbol Device:Battery
- removed C1: 220µF 25V 105°C, symbol My_Device:C_Polarized_Small
- removed C2, C3, C4, C6: 10µF 25V X5R, symbol My_Device:C_Small
- removed C5: 0.1µF 10V X5R, symbol My_Device:C_Small
- removed J1, J2: Conn_01x02, symbol My_Connector_Generic:Conn_01x02
- removed J4: Conn_02x15_Odd_Even, symbol My_Connector_Generic:Conn_02x15_Odd_Even
- removed MD1: OKL-T_6-W12N-C, OKL-T_6-W12N-C:MURATA_OKL-T-6-W12N-C_0, symbol My_Converter_DCDC:OKL-T_6-W12N-C
- removed Q1: Q_PMOS, symbol Device:Q_PMOS
- removed Q2: Q_NMOS, symbol My_Device:Q_NMOS
- removed R1, R2, R3, R6, R7, R8: 10K 1/4W, symbol My_Device:R_Small
- removed R4: 5.1K 1/4W, symbol My_Device:R_Small
- removed R5: 1.2K 1/10W ±1%, symbol My_Device:R_Small
- removed SW1: SW_Slide_2C, symbol My_Switch:SW_Slide_2C
- removed U1: TPS562200DDCR, Package_TO_SOT_SMD:TSOT-23-6, symbol My_Converter_DCDC:TPS562200DDCR
Connections:
- no-connect marks 8 -> 0
Other:
- added sheet ArmUnitBoard (armunit_board.kicad_sch)
- added sheet BatteryBoard (battery_board.kicad_sch)
- added sheet LegUnitBoard (legunit_board.kicad_sch)
- added sheet MainBoard (main_board.kicad_sch)
- note removed: "10kΩ:5.1kΩ = x : 8.4V - x x = 2.837V BATSEN: 0~2.837V"
- note removed: "18350バッテリ 3.7V(MAX 4.7V) 3A 1400mAh"
- note removed: "3.3V"
- note removed: "5V"
- note removed: "7.4V(MAX 8.4V)"
- note removed: "8.4V / 2 / 10kOhm = 0.42mA 0.42mA ^2 * 10kOhm = 0.001764W"
- note removed: "BAT"
- note removed: "EN/RST"
- note removed: "G0/I2S_LRCK/PDM_CLK"
- note removed: "G1/TXD0"
- note removed: "G13/RXD2"
- note removed: "G14/TXD2"
- note removed: "G18/SCK"
- note removed: "G19/GPIO"
- note removed: "G2/I2S_DOUT"
- note removed: "G21/intSDA"
- note removed: "G22/intSCL"
- note removed: "G23/MOSI"
- note removed: "G25/DAC"
- note removed: "G26/DAC"
- note removed: "G27/GPIO"
- note removed: "G3/RXD0"
- note removed: "G32/PA_SDA"
- note removed: "G33/PA_SCL"
- note removed: "G34/PDM_DAT"
- note removed: "G35/ADC"
- note removed: "G36/ADC"
- note removed: "G38/MISO"
- note removed: "GND"
- note removed: "NC"
- note removed: "Rtrim(kOhm) = 5.91 / (Vout - 0.591) = 5.91 / (5.5 - 0.591) = 1.203 kOhm"

Commit message: electric circut complete
Other:
- removed sheet ArmUnitBoard
- removed sheet BatteryBoard
- removed sheet LegUnitBoard
- removed sheet MainBoard
Changed lines of the file:
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@@
 	(generator_version "10.0")
 	(paper "A4")
-	(sheet
-		(at 19.05 17.78)
-		(size 60.96 45.72)
-		(exclude_from_sim no)
-		(in_bom yes)
-		(on_board yes)
-		(dnp no)
-		(fields_autoplaced yes)
-		(stroke
-			(width 0.1524)
-			(type solid)
-		)
-		(fill
-			(color 0 0 0 0)
-		)
-		(property "Sheetname" "BatteryBoard"
-			(at 19.05 17.0684 0)
-			(show_name no)
-			(do_not_autoplace no)
-			(effects
-				(font
-					(size 1.27 1.27)
-				)
-				(justify left bottom)
-			)
-		)
-		(property "Sheetfile" "battery_board.kicad_sch"
-			(at 19.05 64.0846 0)
-			(show_name no)
-			(do_not_autoplace no)
-			(effects
-				(font
-					(size 1.27 1.27)
-				)
-				(justify left top)
-			)
-		)
-		(instances
-			(project "custack-electric"
-				(path "/8000b538-fd6e-48aa-8d1f-0d9d6e323dc5"
-					(page "2")
-				)
-			)
-		)
-	)
-	(sheet
-		(at 97.79 17.78)
-		(size 60.96 44.45)
-		(exclude_from_sim no)
-		(in_bom yes)
-		(on_board yes)
-		(dnp no)
-		(fields_autoplaced yes)
-		(stroke
-			(width 0.1524)
-			(type solid)
-		)
-		(fill
-			(color 0 0 0 0)
-		)
-		(property "Sheetname" "MainBoard"
-			(at 97.79 17.0684 0)
-			(show_name no)
-			(do_not_autoplace no)
-			(effects
-				(font
-					(size 1.27 1.27)
-				)
-				(justify left bottom)
-			)
-		)
-		(property "Sheetfile" "main_board.kicad_sch"
-			(at 97.79 62.8146 0)
-			(show_name no)
-			(do_not_autoplace no)
-			(effects
-				(font
-					(size 1.27 1.27)
-				)
-				(justify left top)
-			)
-		)
-		(instances
-			(project "custack-electric"
-				(path "/8000b538-fd6e-48aa-8d1f-0d9d6e323dc5"
-					(page "3")
-				)
-			)
-		)
-	)
-	(sheet
-		(at 172.72 17.78)
-		(size 59.69 41.91)
-		(exclude_from_sim no)
-		(in_bom yes)
-		(on_board yes)
-		(dnp no)
-		(fields_autoplaced yes)
-		(stroke
-			(width 0.1524)
-			(type solid)
-		)
-		(fill
-			(color 0 0 0 0)
-		)
-		(property "Sheetname" "LegUnitBoard"
-			(at 172.72 17.0684 0)
-			(show_name no)
-			(do_not_autoplace no)
-			(effects
-				(font
-					(size 1.27 1.27)
-				)
-				(justify left bottom)
-			)
-		)
-		(property "Sheetfile" "legunit_board.kicad_sch"
-			(at 172.72 60.2746 0)
-			(show_name no)
-			(do_not_autoplace no)
-			(effects
-				(font
-					(size 1.27 1.27)
-				)
-				(justify left top)
-			)
-		)
-		(instances
-			(project "custack-electric"
-				(path "/8000b538-fd6e-48aa-8d1f-0d9d6e323dc5"
-					(page "4")
-				)
-			)
-		)
-	)
-	(sheet
-		(at 172.72 72.39)
-		(size 59.69 45.72)
-		(exclude_from_sim no)
-		(in_bom yes)
-		(on_board yes)
-		(dnp no)
-		(fields_autoplaced yes)
-		(stroke
-			(width 0.1524)
-			(type solid)
-		)
-		(fill
-			(color 0 0 0 0)
-		)
-		(property "Sheetname" "ArmUnitBoard"
-			(at 172.72 71.6784 0)
-			(show_name no)
-			(do_not_autoplace no)
-			(effects
-				(font
-					(size 1.27 1.27)
-				)
-				(justify left bottom)
-			)
-		)
-		(property "Sheetfile" "armunit_board.kicad_sch"
-			(at 172.72 118.6946 0)
-			(show_name no)
-			(do_not_autoplace no)
-			(effects
-				(font
-					(size 1.27 1.27)
-				)
-				(justify left top)
-			)
-		)
-		(instances
-			(project "custack-electric"
-				(path "/8000b538-fd6e-48aa-8d1f-0d9d6e323dc5"
-					(page "5")
-				)
-			)
-		)
-	)
 	(sheet_instances
 		(path "/"
