File: custack-hardware/electric/leftarmunit_board.kicad_sch (KiCad schematic)
At the start: 18 parts, among them J16 4P MMale magnetic connector (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, J17 PH 2mmピッチ 3極 オス AWG24, J18 PH 2mmピッチ 2極 オス AWG24, Q4 N-ch 30V 4A SOT23F, U10 20MHz 16KB FLASH, U11 Vin(MAX): 13.2V, Vout: 3.3V 2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

Commit message: electric circuit complete
Parts:
- removed C20: 10µF 25V X5R 0603, Capacitor_SMD:C_0603_1608Metric, symbol My_Device:C_Small
- removed C21: 220µF 25V 105°C, Capacitor_SMD:CP_Elec_8x10, symbol My_Device:C_Polarized_Small
- added C20: 100µF 16V 105°C, Capacitor_SMD:CP_Elec_5x5.9, symbol My_Device:C_Polarized_Small
- J16: footprint Connector_PinHeader_2.54mm:PinHeader_1x04_P2.54mm_Vertical -> My_Custom:Pogopin_1x4_2.54mm
Connections:
- net GND: now also C20.2
- net VDD: now also C20.1
Changed lines of the file:
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@@
-	)
-	(junction
-		(at 49.53 72.39)
-		(diameter 0)
-		(color 0 0 0 0)
 	)
 	(junction
@@
 	(wire
 		(pts
-			(xy 41.91 74.93) (xy 41.91 72.39)
-		)
-		(stroke
-			(width 0)
-			(type default)
-		)
-	)
-	(wire
-		(pts
 			(xy 72.39 80.01) (xy 72.39 86.36)
 		)
@@
 	(wire
 		(pts
-			(xy 41.91 80.01) (xy 41.91 83.82)
-		)
-		(stroke
-			(width 0)
-			(type default)
-		)
-	)
-	(wire
-		(pts
 			(xy 163.83 87.63) (xy 171.45 87.63)
 		)
@@
 	(wire
 		(pts
-			(xy 49.53 72.39) (xy 49.53 88.9)
+			(xy 49.53 67.31) (xy 49.53 88.9)
 		)
 		(stroke
@@
 	(wire
 		(pts
-			(xy 49.53 67.31) (xy 49.53 72.39)
-		)
-		(stroke
-			(width 0)
-			(type default)
-		)
-	)
-	(wire
-		(pts
 			(xy 80.01 80.01) (xy 80.01 86.36)
 		)
@@
 		(pts
 			(xy 44.45 151.13) (xy 49.53 151.13)
-		)
-		(stroke
-			(width 0)
-			(type default)
-		)
-	)
-	(wire
-		(pts
-			(xy 41.91 72.39) (xy 49.53 72.39)
 		)
 		(stroke
@@
 			)
 			(justify right bottom)
-		)
-	)
-	(label "GND"
-		(at 41.91 83.82 0)
-		(effects
-			(font
-				(size 1.27 1.27)
-			)
-			(justify left bottom)
 		)
 	)
@@
 	)
 	(symbol
+		(lib_id "My_Device:C_Polarized_Small")
+		(at 95.25 39.37 0)
+		(unit 1)
+		(body_style 1)
+		(exclude_from_sim no)
+		(in_bom yes)
+		(on_board yes)
+		(in_pos_files yes)
+		(dnp no)
+		(fields_autoplaced yes)
+		(property "Reference" "C20"
+			(at 97.79 36.2838 0)
+			(show_name no)
+			(do_not_autoplace no)
+			(effects
+				(font
+					(size 1.016 1.016)
+				)
+				(justify left)
+			)
+		)
+		(property "Value" "100µF 16V 105°C"
+			(at 97.79 38.8238 0)
+			(show_name no)
+			(do_not_autoplace no)
+			(effects
+				(font
+					(size 1.016 1.016)
+				)
+				(justify left)
+			)
+		)
+		(property "Footprint" "Capacitor_SMD:CP_Elec_5x5.9"
+			(at 95.25 39.37 0)
+			(hide yes)
+			(show_name no)
+			(do_not_autoplace no)
+			(effects
+				(font
+					(size 1.27 1.27)
+				)
+			)
+		)
+		(property "Datasheet" "https://www.nichicon.co.jp/english/series_items/catalog_pdf/e-ucm.pdf"
+			(at 95.25 39.37 0)
+			(hide yes)
+			(show_name no)
+			(do_not_autoplace no)
+			(effects
+				(font
+					(size 1.27 1.27)
+				)
+			)
+		)
+		(property "Description" "アルミ電解コンデンサ 100 µF 16 V ラジアル、CAN - SMD 2000時間 @ 105°C"
+			(at 95.25 39.37 0)
+			(hide yes)
+			(show_name no)
+			(do_not_autoplace no)
+			(effects
+				(font
+					(size 1.27 1.27)
+				)
+			)
+		)
+		(property "型式" "UCM1C101MCL1GS"
+			(at 97.79 41.3638 0)
+			(show_name no)
+			(do_not_autoplace no)
+			(effects
+				(font
+					(size 1.016 1.016)
+				)
+				(justify left)
+			)
+		)
+		(pin "2"
+		)
+		(pin "1"
+		)
+		(instances
+			(project "custack-electric"
+				(path "/34724ce1-230f-4531-b3b7-d1c9082b67f0"
+					(reference "C20")
+					(unit 1)
+				)
+			)
+		)
+	)
+	(symbol
 		(lib_id "My_Device:D")
 		(at 133.35 33.02 90)
@@
 	)
 	(symbol
-		(lib_id "My_Device:C_Polarized_Small")
-		(at 95.25 39.37 0)
-		(unit 1)
-		(body_style 1)
-		(exclude_from_sim no)
-		(in_bom yes)
-		(on_board yes)
-		(in_pos_files yes)
-		(dnp no)
-		(fields_autoplaced yes)
-		(property "Reference" "C21"
-			(at 97.79 36.2838 0)
-			(show_name no)
-			(do_not_autoplace no)
-			(effects
-				(font
-					(size 1.016 1.016)
-				)
-				(justify left)
-			)
-		)
-		(property "Value" "220µF 25V 105°C"
-			(at 97.79 38.8238 0)
-			(show_name no)
-			(do_not_autoplace no)
-			(effects
-				(font
-					(size 1.016 1.016)
-				)
-				(justify left)
-			)
-		)
-		(property "Footprint" "Capacitor_SMD:CP_Elec_8x10"
-			(at 95.25 39.37 0)
-			(hide yes)
-			(show_name no)
-			(do_not_autoplace no)
-			(effects
-				(font
-					(size 1.27 1.27)
-				)
-			)
-		)
-		(property "Datasheet" "https://www.nichicon.co.jp/english/series_items/catalog_pdf/e-uud.pdf"
-			(at 95.25 39.37 0)
-			(hide yes)
-			(show_name no)
-			(do_not_autoplace no)
-			(effects
-				(font
-					(size 1.27 1.27)
-				)
-			)
-		)
-		(property "Description" "Polarized capacitor, small symbol"
-			(at 95.25 39.37 0)
-			(hide yes)
-			(show_name no)
-			(do_not_autoplace no)
-			(effects
-				(font
-					(size 1.27 1.27)
-				)
-			)
-		)
-		(property "型式" "UUD1E221MNL1GS"
-			(at 97.79 41.3638 0)
-			(show_name no)
-			(do_not_autoplace no)
-			(effects
-				(font
-					(size 1.016 1.016)
-				)
-				(justify left)
-			)
-		)
-		(pin "2"
-		)
-		(pin "1"
-		)
-		(instances
-			(project "custack-electric"
-				(path "/34724ce1-230f-4531-b3b7-d1c9082b67f0"
-					(reference "C21")
-					(unit 1)
-				)
-			)
-		)
-	)
-	(symbol
 		(lib_id "My_Device:R_Small")
 		(at 80.01 88.9 180)
@@
 			)
 		)
-		(property "Footprint" "Connector_PinHeader_2.54mm:PinHeader_1x04_P2.54mm_Vertical"
+		(property "Footprint" "My_Custom:Pogopin_1x4_2.54mm"
 			(at 30.48 41.91 0)
 			(hide yes)
@@
 			)
 		)
-		(property "Description" "1 セット/5 セット磁気コネクタ 2/3/4/5/6/8 ピンボンディングワイヤーストリップ配線端子強力な磁気無はんだクイックバットジョイント"
+		(property "Description" "Generic connector, single row, 01x04, script generated (kicad-library-utils/schlib/autogen/connector/)"
 			(at 30.48 41.91 0)
 			(hide yes)
@@
 					(unit 1)
 				)
-			)
-		)
-	)
-	(symbol
-		(lib_id "My_Device:C_Small")
-		(at 41.91 77.47 0)
-		(unit 1)
-		(body_style 1)
-		(exclude_from_sim no)
-		(in_bom yes)
-		(on_board yes)
-		(in_pos_files yes)
-		(dnp no)
-		(fields_autoplaced yes)
-		(property "Reference" "C20"
-			(at 39.37 74.9362 0)
-			(show_name no)
-			(do_not_autoplace no)
-			(effects
-				(font
-					(size 1.016 1.016)
-				)
-				(justify right)
-			)
-		)
-		(property "Value" "10µF 25V X5R 0603"
-			(at 39.37 77.4762 0)
-			(show_name no)
-			(do_not_autoplace no)
-			(effects
-				(font
-					(size 1.016 1.016)
-				)
-				(justify right)
-			)
-		)
-		(property "Footprint" "Capacitor_SMD:C_0603_1608Metric"
-			(at 41.91 77.47 0)
-			(hide yes)
-			(show_name no)
-			(do_not_autoplace no)
-			(effects
-				(font
-					(size 1.27 1.27)
-				)
-			)
-		)
-		(property "Datasheet" "https://www.digikey.jp/ja/products/detail/murata-electronics/GRM188R61E106KA73J/9887674?s=N4IgTCBcDaIOICUCyBGAHGhA2FBRFADFgNICCA7AMwBSIAugL5A"
-			(at 41.91 77.47 0)
-			(hide yes)
-			(show_name no)
-			(do_not_autoplace no)
-			(effects
-				(font
-					(size 1.27 1.27)
-				)
-			)
-		)
-		(property "Description" "Unpolarized capacitor, small symbol"
-			(at 41.91 77.47 0)
-			(hide yes)
-			(show_name no)
-			(do_not_autoplace no)
-			(effects
-				(font
-					(size 1.27 1.27)
-				)
-			)
-		)
-		(property "型式" "GRM188R61E106KA73J"
-			(at 39.37 80.0162 0)
-			(show_name no)
-			(do_not_autoplace no)
-			(effects
-				(font
-					(size 1.016 1.016)
-				)
-				(justify right)
-			)
-		)
-		(pin "1"
-		)
-		(pin "2"
-		)
-		(instances
-			(project "custack-electric"
-				(path "/34724ce1-230f-4531-b3b7-d1c9082b67f0"
-					(reference "C20")
-					(unit 1)
-				)
