File: custack-hardware/electric/legunit_board.kicad_sch (KiCad schematic)
At the start: 25 parts, among them J10 PH 2mmピッチ 3極 オス AWG24, J11 PH 2mmピッチ 3極 オス AWG24, J12 PH 2mmピッチ 3極 オス AWG24, J7 4P MMale magnetic connector (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, J8 PH 2mmピッチ 3極 オス AWG24, J9 PH 2mmピッチ 3極 オス AWG24, U2 20MHz 16KB FLASH, U3 非反転 1.65-5.5V, 32mA SOT-23-5, U4 非反転 1.65-5.5V, 32mA SOT-23-5, U5 Vin(MAX): 13.2V, Vout: 3.3V 2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, U6 非反転 1.65-5.5V, 32mA SOT-23-5, U7 非反転 1.65-5.5V, 32mA SOT-23-5

Commit message: 電気回路の修正
Connections:
- net EXT_SCA is gone; now on net EXT_SCL: J7.3 (Pin_3), R19.1, U2.12 (PA2)
- net EXT_SCL: no longer J7.4 (Pin_4), R20.1, U2.11 (PA1)
- new net EXT_SDA: J7.4 (Pin_4), R20.1, U2.11 (PA1)
Changed lines of the file:
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@@
 		)
 	)
-	(label "EXT_SCL"
+	(label "EXT_SDA"
 		(at 96.52 101.6 180)
 		(effects
@@
 		)
 	)
-	(label "EXT_SCA"
+	(label "EXT_SCL"
 		(at 53.34 38.1 180)
 		(effects
@@
 		)
 	)
-	(label "EXT_SCL"
+	(label "EXT_SDA"
 		(at 53.34 35.56 180)
 		(effects
@@
 		)
 	)
-	(label "EXT_SCA"
+	(label "EXT_SCL"
 		(at 96.52 99.06 180)
 		(effects
