File: custack-hardware/electric/rightarmunit_board.kicad_sch (KiCad schematic)
At the start: 18 parts, among them J13 4P MMale magnetic connector (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, J14 PH 2mmピッチ 3極 オス AWG24, J15 PH 2mmピッチ 2極 オス AWG24, Q3 N-ch 30V 4A SOT23F, U8 20MHz 16KB FLASH, U9 Vin(MAX): 13.2V, Vout: 3.3V 2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

Commit message: electric circuit complete
Parts:
- removed C16: 10µF 25V X5R 0603, Capacitor_SMD:C_0603_1608Metric, symbol My_Device:C_Small
- C17: value 220µF 25V 105°C -> 100µF 16V 105°C; footprint Capacitor_SMD:CP_Elec_8x10 -> Capacitor_SMD:CP_Elec_5x5.9; 型式 UUD1E221MNL1GS -> UCM1C101MCL1GS
- J13: footprint Connector_PinHeader_2.54mm:PinHeader_1x04_P2.54mm_Vertical -> My_Custom:Pogopin_1x4_2.54mm
