File: custack-hardware/electric/rightarmunit_board.kicad_sch (KiCad schematic)
At the start: 17 parts, among them J13 4P MMale magnetic connector (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, J14 PH 2mmピッチ 3極 オス AWG24, J15 PH 2mmピッチ 2極 オス AWG24, Q3 N-ch 30V 4A SOT23F, U8 20MHz 16KB FLASH, U9 Vin(MAX): 13.2V, Vout: 3.3V 2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

Commit message: 電気回路の修正
Connections:
- net EXT_SCA is gone; now on net EXT_SCL: J13.3 (Pin_3), R26.1, U8.12 (PA2)
- net EXT_SCL: no longer J13.4 (Pin_4), R27.1, U8.11 (PA1)
- new net EXT_SDA: J13.4 (Pin_4), R27.1, U8.11 (PA1)
Changed lines of the file:
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@@
 		)
 	)
-	(label "EXT_SCA"
+	(label "EXT_SCL"
 		(at 48.26 39.37 180)
 		(effects
@@
 		)
 	)
-	(label "EXT_SCA"
+	(label "EXT_SCL"
 		(at 91.44 99.06 180)
 		(effects
@@
 		)
 	)
-	(label "EXT_SCL"
+	(label "EXT_SDA"
 		(at 91.44 101.6 180)
 		(effects
@@
 		)
 	)
-	(label "EXT_SCL"
+	(label "EXT_SDA"
 		(at 48.26 36.83 180)
 		(effects
