File: custack-hardware/electric/custack-electric.kicad_pcb (KiCad board)
At the start: 2 copper layers, 92 x 62.9 mm, 105 parts, among them J1 XH 2.5mmピッチ 2極 オス AWG22, J10 PH 2mmピッチ 3極 オス AWG24, J11 PH 2mmピッチ 3極 オス AWG24, J12 PH 2mmピッチ 3極 オス AWG24, J13 4P MMale magnetic connector (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, J14 PH 2mmピッチ 3極 オス AWG24, J15 PH 2mmピッチ 2極 オス AWG24, J16 4P MMale magnetic connector (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, J17 PH 2mmピッチ 3極 オス AWG24, J18 PH 2mmピッチ 2極 オス AWG24, J2 XH 2.5mmピッチ 2極 オス AWG24, J3 2x15P@2.54mm SMD, J4 PH 2mmピッチ 4極 オス AWG24, J5 PH 2mmピッチ 4極 オス AWG24, J6 PH 2mmピッチ 4極 オス AWG24, J7 4P MMale magnetic connector (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, J8 PH 2mmピッチ 3極 オス AWG24, J9 PH 2mmピッチ 3極 オス AWG24, Q1 MOSFET P-CH 20V 6A SOT23F, Q2 N-ch 30V 4A SOT23F, Q3 N-ch 30V 4A SOT23F, Q4 N-ch 30V 4A SOT23F, SW1 12V 100mA, U1 IN:4.5V-17V, OUT:0.765V-7V,2A, U10 20MHz 16KB FLASH, U11 Vin(MAX): 13.2V, Vout: 3.3V 2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, U2 20MHz 16KB FLASH, U3 非反転 1.65-5.5V, 32mA SOT-23-5, U4 非反転 1.65-5.5V, 32mA SOT-23-5, U5 Vin(MAX): 13.2V, Vout: 3.3V 2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, U6 非反転 1.65-5.5V, 32mA SOT-23-5, U7 非反転 1.65-5.5V, 32mA SOT-23-5, U8 20MHz 16KB FLASH, U9 Vin(MAX): 13.2V, Vout: 3.3V 2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

Commit message: electric circuit complete
Parts:
- removed C12, C16: 10µF 25V X5R 0603, Capacitor_SMD:C_0603_1608Metric
- removed C21: 220µF 25V 105°C, Capacitor_SMD:CP_Elec_8x10
- C13, C17: value 220µF 25V 105°C -> 100µF 16V 105°C; footprint Capacitor_SMD:CP_Elec_8x10 -> Capacitor_SMD:CP_Elec_5x5.9
- C20: value 10µF 25V X5R 0603 -> 100µF 16V 105°C; footprint Capacitor_SMD:C_0603_1608Metric -> Capacitor_SMD:CP_Elec_5x5.9
- J13, J16, J7: footprint Connector_PinHeader_2.54mm:PinHeader_1x04_P2.54mm_Vertical -> My_Custom:Pogopin_1x4_2.54mm; moved to B.Cu
- moved U10 163.8 mm to (88.7, 89.5), turned to 90 degrees
- moved Q4 160.5 mm to (88.7, 80.5), turned to 90 degrees
- moved D12 158.0 mm to (86.5, 77.0)
- moved U11 155.9 mm to (97.0, 91.0), turned to 180 degrees
- moved J18 153.0 mm to (86.5, 72.0)
- moved J16 152.6 mm to (95.4, 82.5), turned to 180 degrees
- moved D9 145.8 mm to (98.0, 79.0)
- moved R26 144.9 mm to (66.5, 86.5), turned to -90 degrees
- moved U8 144.8 mm to (76.0, 89.5), turned to 90 degrees
- moved R32 144.7 mm to (88.7, 84.0), turned to -90 degrees
- moved D6 143.9 mm to (61.0, 91.5), turned to 180 degrees
- moved D7 142.4 mm to (61.0, 88.5), turned to 180 degrees
- moved R27 142.2 mm to (68.5, 86.5), turned to -90 degrees
- moved R29 141.7 mm to (91.7, 78.5), turned to -90 degrees
- moved D10 140.1 mm to (103.7, 92.0)
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Connections:
- C20 pad 1: /leftarmunit_board/+3.3V -> /leftarmunit_board/VDD
Routing:
- net /legunit_board/EXT_SCL: track 0.00 -> 25.0 mm, vias 0 -> 2
- net /leftarmunit_board/VBUS: track 0.00 -> 22.6 mm
- net /rightarmunit_board/VBUS: track 0.00 -> 22.0 mm
- net /legunit_board/EXT_SCA: track 0.00 -> 20.3 mm, vias 0 -> 2
- net /leftarmunit_board/PWM1: track 0.00 -> 20.0 mm
- net /legunit_board/PWM1: track 0.00 -> 19.2 mm
- net Net-(J8-Pin_3): track 0.00 -> 18.3 mm
- net Net-(J14-Pin_3): track 0.00 -> 17.9 mm, vias 0 -> 1
- net /legunit_board/PWM2: track 0.00 -> 15.6 mm
- net Net-(J17-Pin_3): track 0.00 -> 15.4 mm, vias 0 -> 1
- net /leftarmunit_board/EXT_SCA: track 0.00 -> 15.3 mm, vias 0 -> 1
- net Net-(J9-Pin_1): track 0.00 -> 13.2 mm
- net Net-(J11-Pin_1): track 0.00 -> 13.0 mm
- net /rightarmunit_board/PWM1: track 0.00 -> 12.8 mm, vias 0 -> 2
- net /leftarmunit_board/+3.3V: track 0.00 -> 12.5 mm
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- added copper zone on F.Cu, net /leftarmunit_board/+3.3V
- added copper zone on B.Cu, net /leftarmunit_board/GND
- added copper zone on F.Cu, net /leftarmunit_board/GND
- added copper zone on B.Cu, net /leftarmunit_board/VDD
- added copper zone on F.Cu, net /leftarmunit_board/VDD
- added copper zone on B.Cu, net /legunit_board/+3.3V
- added copper zone on F.Cu, net /legunit_board/+3.3V
- added copper zone on B.Cu, net /legunit_board/GND
- added copper zone on F.Cu, net /legunit_board/GND
- added copper zone on B.Cu, net /legunit_board/VDD
- added copper zone on F.Cu, net /legunit_board/VDD
- added copper zone on F.Cu, net /rightarmunit_board/+3.3V
- added copper zone on B.Cu, net /rightarmunit_board/GND
- added copper zone on F.Cu, net /rightarmunit_board/GND
- added copper zone on F.Cu, net /rightarmunit_board/VDD
- added copper zone on F.Cu, net Net-(D10-K)
- added copper zone on F.Cu, net Net-(D12-A)
- added copper zone on F.Cu, net Net-(D3-K)
- added copper zone on F.Cu, net Net-(D6-K)
- added copper zone on F.Cu, net Net-(D8-A)
Other:
- board size 92 x 62.9 mm -> 92 x 65 mm

Commit message: pcb board complete
Parts:
- added REF**: MouseBite-Slot_2.0x4.5mm_outset_D0.5mm_P0.85mm_7h, Panelization:MouseBite-Slot_2.0x4.5mm_outset_D0.5mm_P0.85mm_7h, F.Cu at (82.0, 81.5)
- added REF**: MountingHole_2.1mm, MountingHole:MountingHole_2.1mm, F.Cu at (21.5, 108.5)
- added REF**: MouseBite-Slot_2.0x4.5mm_outset_D0.5mm_P0.85mm_7h, Panelization:MouseBite-Slot_2.0x4.5mm_outset_D0.5mm_P0.85mm_7h, F.Cu at (26.0, 74.0)
- added REF**: MouseBite-Slot_2.0x4.5mm_outset_D0.5mm_P0.85mm_7h, Panelization:MouseBite-Slot_2.0x4.5mm_outset_D0.5mm_P0.85mm_7h, F.Cu at (31.6, 66.5)
- added REF**: Fiducial_1mm_Mask2mm, Fiducial:Fiducial_1mm_Mask2mm, F.Cu at (22.9, 104.0)
- added REF**: MouseBite-Slot_2.0x4.5mm_outset_D0.5mm_P0.85mm_7h, Panelization:MouseBite-Slot_2.0x4.5mm_outset_D0.5mm_P0.85mm_7h, F.Cu at (96.0, 81.5)
- added REF**: MouseBite-Slot_2.0x4.5mm_outset_D0.5mm_P0.85mm_7h, Panelization:MouseBite-Slot_2.0x4.5mm_outset_D0.5mm_P0.85mm_7h, F.Cu at (26.0, 61.0)
- added REF**: Fiducial_1mm_Mask2mm, Fiducial:Fiducial_1mm_Mask2mm, F.Cu at (104.7, 104.0)
- added REF**: MouseBite-Slot_2.0x4.5mm_outset_D0.5mm_P0.85mm_7h, Panelization:MouseBite-Slot_2.0x4.5mm_outset_D0.5mm_P0.85mm_7h, F.Cu at (101.5, 35.0)
- added REF**: MouseBite-Slot_2.0x4.5mm_outset_D0.5mm_P0.85mm_7h, Panelization:MouseBite-Slot_2.0x4.5mm_outset_D0.5mm_P0.85mm_7h, F.Cu at (71.5, 89.0)
- added REF**: MouseBite-Slot_2.0x4.5mm_outset_D0.5mm_P0.85mm_7h, Panelization:MouseBite-Slot_2.0x4.5mm_outset_D0.5mm_P0.85mm_7h, F.Cu at (76.5, 35.0)
- added REF**: MouseBite-Slot_2.0x4.5mm_outset_D0.5mm_P0.85mm_7h, Panelization:MouseBite-Slot_2.0x4.5mm_outset_D0.5mm_P0.85mm_7h, F.Cu at (101.5, 62.0)
- added REF**: MouseBite-Slot_2.0x4.5mm_outset_D0.5mm_P0.85mm_7h, Panelization:MouseBite-Slot_2.0x4.5mm_outset_D0.5mm_P0.85mm_7h, F.Cu at (26.0, 35.0)
- added REF**: MouseBite-Slot_2.0x4.5mm_outset_D0.5mm_P0.85mm_7h, Panelization:MouseBite-Slot_2.0x4.5mm_outset_D0.5mm_P0.85mm_7h, F.Cu at (101.5, 105.0)
- added REF**: MountingHole_2.1mm, MountingHole:MountingHole_2.1mm, F.Cu at (106.0, 108.5)
- added REF**: MouseBite-Slot_2.0x4.5mm_outset_D0.5mm_P0.85mm_7h, Panelization:MouseBite-Slot_2.0x4.5mm_outset_D0.5mm_P0.85mm_7h, F.Cu at (71.5, 99.5)
- added REF**: Fiducial_1mm_Mask2mm, Fiducial:Fiducial_1mm_Mask2mm, F.Cu at (104.7, 36.5)
- added REF**: MountingHole_2.1mm, MountingHole:MountingHole_2.1mm, F.Cu at (106.0, 32.0)
- added REF**: MountingHole_2.1mm, MountingHole:MountingHole_2.1mm, F.Cu at (21.5, 32.0)
- added REF**: MouseBite-Slot_2.0x4.5mm_outset_D0.5mm_P0.85mm_7h, Panelization:MouseBite-Slot_2.0x4.5mm_outset_D0.5mm_P0.85mm_7h, F.Cu at (101.5, 49.0)
- added REF**: MouseBite-Slot_2.0x4.5mm_outset_D0.5mm_P0.85mm_7h, Panelization:MouseBite-Slot_2.0x4.5mm_outset_D0.5mm_P0.85mm_7h, F.Cu at (101.5, 89.0)
- added REF**: MouseBite-Slot_2.0x4.5mm_outset_D0.5mm_P0.85mm_7h, Panelization:MouseBite-Slot_2.0x4.5mm_outset_D0.5mm_P0.85mm_7h, F.Cu at (76.5, 61.0)
- added REF**: MouseBite-Slot_2.0x4.5mm_outset_D0.5mm_P0.85mm_7h, Panelization:MouseBite-Slot_2.0x4.5mm_outset_D0.5mm_P0.85mm_7h, F.Cu at (61.5, 66.5)
- added REF**: Fiducial_1mm_Mask2mm, Fiducial:Fiducial_1mm_Mask2mm, F.Cu at (22.9, 36.5)
- added REF**: MouseBite-Slot_2.0x4.5mm_outset_D0.5mm_P0.85mm_7h, Panelization:MouseBite-Slot_2.0x4.5mm_outset_D0.5mm_P0.85mm_7h, F.Cu at (101.5, 76.0)
- added REF**: MouseBite-Slot_2.0x4.5mm_outset_D0.5mm_P0.85mm_7h, Panelization:MouseBite-Slot_2.0x4.5mm_outset_D0.5mm_P0.85mm_7h, F.Cu at (26.0, 101.0)
- moved C10 62.6 mm to (47.5, 84.0)
- moved C11 62.6 mm to (55.5, 84.0)
- moved C3 62.6 mm to (43.0, 86.5)
- moved C4 62.6 mm to (43.0, 84.5)
- moved C5 62.6 mm to (40.0, 80.5)
- moved C9 62.6 mm to (36.5, 104.5)
- moved J2 62.6 mm to (48.2, 103.5)
- moved J3 62.6 mm to (30.1, 69.8)
- moved J4 62.6 mm to (66.5, 73.0)
- moved J5 62.6 mm to (66.5, 84.5)
- moved J6 62.6 mm to (66.5, 96.0)
- moved L1 62.6 mm to (35.7, 83.0)
- moved MD1 62.6 mm to (51.5, 92.0)
- moved Q2 62.6 mm to (38.5, 96.0)
- moved R10 62.6 mm to (36.5, 100.5)
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Other:
- board size 92 x 65 mm -> 89.5 x 81.5 mm
