File: custack-hardware/electric/custack-electric.kicad_pcb (KiCad board)
At the start: 2 copper layers, 89.5 x 81.5 mm, 128 parts, among them J1 XH 2.5mmピッチ 2極 オス AWG22, J10 PH 2mmピッチ 3極 オス AWG24, J11 PH 2mmピッチ 3極 オス AWG24, J12 PH 2mmピッチ 3極 オス AWG24, J13 4P MMale magnetic connector (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, J14 PH 2mmピッチ 3極 オス AWG24, J15 PH 2mmピッチ 2極 オス AWG24, J16 4P MMale magnetic connector (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, J17 PH 2mmピッチ 3極 オス AWG24, J18 PH 2mmピッチ 2極 オス AWG24, J2 XH 2.5mmピッチ 2極 オス AWG24, J3 2x15P@2.54mm SMD, J4 PH 2mmピッチ 4極 オス AWG24, J5 PH 2mmピッチ 4極 オス AWG24, J6 PH 2mmピッチ 4極 オス AWG24, J7 4P MMale magnetic connector (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, J8 PH 2mmピッチ 3極 オス AWG24, J9 PH 2mmピッチ 3極 オス AWG24, Q1 MOSFET P-CH 20V 6A SOT23F, Q2 N-ch 30V 4A SOT23F, Q3 N-ch 30V 4A SOT23F, Q4 N-ch 30V 4A SOT23F, SW1 12V 100mA, U1 IN:4.5V-17V, OUT:0.765V-7V,2A, U10 20MHz 16KB FLASH, U11 Vin(MAX): 13.2V, Vout: 3.3V 2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, U2 20MHz 16KB FLASH, U3 非反転 1.65-5.5V, 32mA SOT-23-5, U4 非反転 1.65-5.5V, 32mA SOT-23-5, U5 Vin(MAX): 13.2V, Vout: 3.3V 2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, U6 非反転 1.65-5.5V, 32mA SOT-23-5, U7 非反転 1.65-5.5V, 32mA SOT-23-5, U8 20MHz 16KB FLASH, U9 Vin(MAX): 13.2V, Vout: 3.3V 2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

Commit message: complete electric board design
Parts:
- turned Q1 to -90 degrees
Connections:
- Q1 pad 2: /battery_board/+VSW -> /battery_board/+BATT
- Q1 pad 3: /battery_board/+BATT -> /battery_board/+VSW
Routing:
- net Net-(Q1-G): track 0.00 -> 10.5 mm, vias 0 -> 2
- removed copper zone on F.Cu, net Net-(Q1-G)
